Commit message: enabled slam using cartographer
2D lidar (rplidar a1)
no imu needed

File: catkin_ws/src/main/xacro/dtw_robot.xacro (robot description, xacro)
@@ -22,7 +22,7 @@
     </link>
   </xacro:macro>
-  <link name="world"/>
+  <link name="map"/>
   <joint name="base_joint" type="floating">
-    <parent link="world"/>
+    <parent link="map"/>
     <child  link="base_link"/>
   </joint>

Commit message: joystick to control motors of the 2 wheels

File: catkin_ws/src/main/xacro/dtw_robot.xacro (robot description, xacro)
@@ -6,6 +6,22 @@
     <color rgba="1.0 0.0 0.0 2.5"/>
   </material>
+<!--  <xacro:macro name="wheel_macro" params="parent prefix xyz">-->
+<!--    <joint name="${prefix}_joint" type="continuous">-->
+<!--      <origin xyz="${xyz}" rpy="${radians(-90)} 0 0"/>-->
+<!--      <parent link="${parent}"/>-->
+<!--      <child  link="${prefix}_link"/>-->
+<!--      <axis xyz="0 0 1" />-->
+<!--    </joint>-->
+<!--    <link name="${prefix}_link">-->
+<!--      <visual>-->
+<!--        <geometry>-->
+<!--          <cylinder radius="0.05" length="0.02" />-->
+<!--        </geometry>-->
+<!--        <material name="red"/>-->
+<!--      </visual>-->
+<!--    </link>-->
+<!--  </xacro:macro> -->
   <xacro:macro name="wheel_macro" params="parent prefix xyz">
-    <joint name="${prefix}_joint" type="continuous">
+    <joint name="${prefix}_joint" type="fixed">
       <origin xyz="${xyz}" rpy="${radians(-90)} 0 0"/>
       <parent link="${parent}"/>
